File: Flatbox-rev5.kicad_pcb (KiCad board)
At the start: 2 copper layers, 233.5 x 120 mm, 27 parts, among them SW1 SW_Push, SW10 SW_Push, SW11 SW_Push, SW12 SW_Push, SW13 SW_Push, SW14 SW_Push, SW15 SW_Push, SW16 SW_Push, SW17 SW_Push, SW18 SW_Push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

Commit message: Wiring, but unfilled?
Parts:
- added SW20: SW_Push, Button_Switch_THT:SW_PUSH_6mm_H5mm, F.Cu at (92.7, 33.5)
- moved A1 14.1 mm to (119.0, 32.0)
- moved H1 14.1 mm to (37.0, 27.0)
- moved H4 14.1 mm to (37.0, 153.0)
- moved SW10 14.1 mm to (159.6, 86.6)
- moved SW11 14.1 mm to (186.2, 75.0)
- moved SW12 14.1 mm to (215.1, 74.9)
- moved SW13 14.1 mm to (244.1, 80.3)
- moved SW14 14.1 mm to (154.0, 117.6)
- moved SW15 14.1 mm to (180.6, 106.5)
- moved SW16 14.1 mm to (209.5, 106.5)
- moved SW17 14.1 mm to (238.7, 111.6)
- moved SW19 14.1 mm to (209.5, 43.6)
- moved SW5 14.1 mm to (180.6, 43.6)
- moved SW6 14.1 mm to (154.0, 55.5)
- moved SW7 14.1 mm to (48.2, 75.0)
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Connections:
- A1 pad 1: unconnected-(A1-GPIO0-Pad1) -> L1
- A1 pad 10: CROSS -> SQUARE
- A1 pad 11: UP -> CROSS
- A1 pad 12: RIGHT -> UP
- A1 pad 13: DOWN -> LEFT
- A1 pad 14: LEFT -> DOWN
- A1 pad 15: OPT1 -> RIGHT
- A1 pad 16: OPT2 -> OPT1
- A1 pad 17: OPT3 -> OPT2
- A1 pad 18: OPT4 -> OPT3
- A1 pad 19: L3 -> OPT4
- A1 pad 2: TOUCH -> L2
- A1 pad 20: R3 -> OPT5
- A1 pad 3: L1 -> L3
- A1 pad 4: L2 -> R1
- A1 pad 5: R1 -> R2
- A1 pad 6: R2 -> R3
- A1 pad 9: SQUARE -> TOUCH
- SW19 pad 1: TOUCH -> L3
- SW5 pad 1: L3 -> R3
- SW6 pad 1: R3 -> TOUCH
Routing:
- net L2: track 0.00 -> 221.1 mm
- net L1: track 0.00 -> 190.2 mm
- net R2: track 0.00 -> 183.8 mm
- net R1: track 0.00 -> 152.4 mm
- net CIRCLE: track 0.00 -> 139.4 mm
- net CROSS: track 0.00 -> 122.8 mm
- net L3: track 0.74 -> 121.0 mm
- net TRIANGLE: track 0.00 -> 107.2 mm
- net SQUARE: track 0.00 -> 87.9 mm
- net DOWN: track 64.6 -> 152.3 mm
- net LEFT: track 105.1 -> 187.0 mm
- net R3: track 0.68 -> 74.8 mm
- net TOUCH: track 0.00 -> 54.1 mm
- net RIGHT: track 79.4 -> 113.5 mm
- net OPT5: track 0.00 -> 28.2 mm
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Other:
- board size 233.5 x 120 mm -> 235 x 140 mm
