File: Flatbox-rev5.kicad_pcb (KiCad board)
At the start: 2 copper layers, 235 x 140 mm, 28 parts, among them SW1 SW_Push, SW10 SW_Push, SW11 SW_Push, SW12 SW_Push, SW13 SW_Push, SW14 SW_Push, SW15 SW_Push, SW16 SW_Push, SW17 SW_Push, SW18 SW_Push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

Commit message: Cleaning up unused tracks.
Routing:
- net LEFT: track 187.0 -> 185.5 mm
Changed lines of the file:
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@@
   (segment (start 37 100) (end 37 84) (width 0.254) (layer "F.Cu") (net 2))
   (segment (start 119 102) (end 39 102) (width 0.254) (layer "F.Cu") (net 2))
-  (segment (start 116.46 43.7) (end 116.46 44.54) (width 0.254) (layer "F.Cu") (net 2))
   (segment (start 116.46 43.7) (end 116.46 62.46) (width 0.254) (layer "F.Cu") (net 2))
   (segment (start 121 67) (end 121 100) (width 0.254) (layer "F.Cu") (net 2))
@@
   (segment (start 116.46 62.46) (end 121 67) (width 0.254) (layer "F.Cu") (net 2))
   (segment (start 39 102) (end 37 100) (width 0.254) (layer "F.Cu") (net 2))
-  (segment (start 116.46 44.54) (end 116 45) (width 0.254) (layer "F.Cu") (net 2))
   (segment (start 48.225 80.95) (end 44.95 77.675) (width 0.254) (layer "B.Cu") (net 2))
   (segment (start 44.95 77.675) (end 44.95 69.1) (width 0.254) (layer "B.Cu") (net 2))
