File: Flatbox-rev5.kicad_sch (KiCad schematic)
At the start: 27 parts, among them SW1 SW_Push, SW10 SW_Push, SW11 SW_Push, SW12 SW_Push, SW13 SW_Push, SW14 SW_Push, SW15 SW_Push, SW16 SW_Push, SW17 SW_Push, SW18 SW_Push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

Commit message: Wiring, but unfilled?
Parts:
- added SW20: SW_Push, Button_Switch_THT:SW_PUSH_6mm_H5mm, symbol Switch:SW_Push
Connections:
- net CROSS: now also A1.11 (GPIO10); no longer A1.10 (GPIO9)
- net DOWN: now also A1.14 (GPIO13); no longer A1.13 (GPIO12)
- net GND: now also SW20.2
- net L1: now also A1.1 (GPIO0); no longer A1.3 (GPIO2)
- net L2: now also A1.2 (GPIO1); no longer A1.4 (GPIO3)
- net L3: now also A1.3 (GPIO2), SW19.1; no longer A1.19 (GPIO28), SW5.1
- net LEFT: now also A1.13 (GPIO12); no longer A1.14 (GPIO13)
- net OPT1: now also A1.16 (GPIO15); no longer A1.15 (GPIO14)
- net OPT2: now also A1.17 (GPIO26); no longer A1.16 (GPIO15)
- net OPT3: now also A1.18 (GPIO27); no longer A1.17 (GPIO26)
- net OPT4: now also A1.19 (GPIO28); no longer A1.18 (GPIO27)
- net R1: now also A1.4 (GPIO3); no longer A1.5 (GPIO4)
- net R2: now also A1.5 (GPIO4); no longer A1.6 (GPIO5)
- net R3: now also A1.6 (GPIO5), SW5.1; no longer A1.20 (GPIO29), SW6.1
- net RIGHT: now also A1.15 (GPIO14); no longer A1.12 (GPIO11)
- net SQUARE: now also A1.10 (GPIO9); no longer A1.9 (GPIO8)
- net TOUCH: now also A1.9 (GPIO8), SW6.1; no longer A1.2 (GPIO1), SW19.1
- net UP: now also A1.12 (GPIO11); no longer A1.11 (GPIO10)
- new net OPT5: A1.20 (GPIO29), SW20.1
