File: rabodo.kicad_pcb (KiCad board)
At the start: 2 copper layers, 235 x 140 mm, 28 parts, among them SW1 SW_Push, SW10 SW_Push, SW11 SW_Push, SW12 SW_Push, SW13 SW_Push, SW14 SW_Push, SW15 SW_Push, SW16 SW_Push, SW17 SW_Push, SW18 SW_Push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

Commit message: Renaming!
Parts:
- added G***: LOGO, LOGO, F.Cu at (69.0, 123.0)
Routing:
- net UP: track 156.5 -> 159.0 mm
Other:
- board text added: "github.com/acedio/rabodo"
- board text added: "rabodo"
- board text added: "rev1"
- board text removed: "Fatbox"
- board text removed: "github.com/jfedor2/flatbox"
- board text removed: "rev5"

Commit message: Expanding and rewiring board.
Parts:
- added H10: MountingHole, MountingHole:MountingHole_6.4mm_M6, F.Cu at (305.0, 110.0)
- added H8: MountingHole, MountingHole:MountingHole_6.4mm_M6, F.Cu at (215.0, 35.0)
- added H9: MountingHole, MountingHole:MountingHole_6.4mm_M6, F.Cu at (35.0, 110.0)
- moved H7 97.4 mm to (125.0, 185.0)
- moved H5 72.4 mm to (215.0, 185.0)
- moved H6 56.9 mm to (305.0, 185.0)
- moved A1 50.0 mm to (169.0, 32.0)
- moved H3 47.7 mm to (305.0, 35.0)
- moved H4 32.1 mm to (35.0, 185.0)
- moved SW17 32.0 mm to (263.7, 131.6)
- moved SW10 32.0 mm to (184.6, 106.6)
- moved SW11 32.0 mm to (211.2, 95.0)
- moved SW12 32.0 mm to (240.1, 94.9)
- moved SW13 32.0 mm to (269.1, 100.3)
- moved SW14 32.0 mm to (179.0, 137.6)
- moved SW15 32.0 mm to (205.6, 126.5)
- moved SW16 32.0 mm to (234.5, 126.5)
- moved SW19 32.0 mm to (234.5, 63.6)
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Routing:
- net OPT5: track 28.2 -> 77.0 mm
- net OPT2: track 57.6 -> 106.3 mm
- net OPT4: track 38.0 -> 86.7 mm
- net OPT3: track 47.8 -> 96.5 mm
- net OPT1: track 67.3 -> 116.1 mm
- net UP: track 159.0 -> 186.9 mm
- net LEFT: track 185.5 -> 212.1 mm
- net DOWN: track 152.3 -> 177.6 mm
- net RIGHT: track 113.5 -> 137.3 mm
- net R2: track 183.8 -> 160.5 mm
- net R1: track 152.4 -> 129.1 mm
- net L3: track 121.0 -> 97.7 mm
- net L1: track 190.2 -> 166.9 mm
- net L2: track 221.1 -> 197.7 mm
- net TOUCH: track 54.1 -> 73.8 mm
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Other:
- board size 235 x 140 mm -> 300 x 180 mm
