File: rabodo.kicad_pcb (KiCad board)
At the start: 2 copper layers, 300 x 180 mm, 32 parts, among them SW1 SW_Push, SW10 SW_Push, SW11 SW_Push, SW12 SW_Push, SW13 SW_Push, SW14 SW_Push, SW15 SW_Push, SW16 SW_Push, SW17 SW_Push, SW18 SW_Push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

Commit message: Updating to fill the front of the PCB with a ground plane and widening the traces + spacing.
Routing:
- net OPT1: track 116.1 -> 121.0 mm
- net OPT2: track 106.3 -> 110.4 mm
- net L1: track 166.9 -> 171.0 mm
- net GND: track 4.00 -> 0.00 mm, vias 1 -> 0
- net L2: track 197.7 -> 201.2 mm
- net OPT3: track 96.5 -> 99.8 mm
- net RIGHT: track 137.3 -> 134.6 mm
- net OPT4: track 86.7 -> 89.2 mm
- net UP: track 186.9 -> 185.1 mm
- net OPT5: track 77.0 -> 78.6 mm
- net CROSS: track 134.6 -> 136.2 mm
- net R2: track 160.5 -> 159.3 mm
- net CIRCLE: track 135.6 -> 134.4 mm
- net TRIANGLE: track 103.3 -> 102.2 mm
- net R1: track 129.1 -> 127.9 mm
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- added copper zone on F.Cu, net GND
Other:
- board text removed: "RP2040-Zero"
